File: kicad/esp32_pcb/esp32_pcb.kicad_sch (KiCad schematic)
At the start: 0 parts

Commit message: Added basic voltage regulations
Added a 5v voltage regulator for the external electronics and added a 3.3v one for the ESP32. Also added a 0.1uF and 1uF decoupled capacitors on VDD_SPI pins on ESP32.
Parts:
- added 0.1uF: 0.1uF, symbol Device:C
- added 1uF: 1uF, symbol Device:C
- added U1: ESP32-S3, Package_DFN_QFN:QFN-56-1EP_7x7mm_P0.4mm_EP4x4mm, symbol MCU_Espressif:ESP32-S3
- added U2: L7805, symbol Regulator_Linear:L7805
- added U3: LD1117V33, Package_TO_SOT_THT:TO-220-3_Vertical, symbol Regulator_Linear:LD1117V33
Connections:
- new net: 0.1uF.2, 1uF.2, U1.46 (VDD3P3_CPU)
- new net: U1.2 (VDD3P3), U1.20 (VDD3P3_RTC), U1.29 (VDD_SPI), U1.3 (VDD3P3), U1.55 (VDDA), U1.56 (VDDA), U3.2 (VO)
- new net +5V: U2.1 (IN), U3.3 (VI)
- new net GND: 0.1uF.1, 1uF.1, U1.57 (GND), U2.2 (GND), U3.1 (GND)

Commit message: Added stuff to the pcb
Parts:
- added D1: Power, symbol Device:LED
- added D3: LED_ARGB, symbol Device:LED_ARGB
- added R1, R3, R4, R5: R, symbol Device:R
Connections:
- net GND: now also D1.1 (K), D3.1 (A)
- net at U2.3 (OUT): now also R1.2
- new net: D1.2 (A), R1.1
- new net: D3.3 (GK), R4.2
- new net: D3.2 (RK), R3.2
- new net: D3.4 (BK), R5.2
